File: electronics/MacroPad SP25 End/MacroPad SP25 End--Long.kicad_pcb (KiCad board)
At the start: 2 copper layers, 72 x 123.5 mm, 16 parts, among them J1 Conn_01x07_Pin, J2 Conn_01x07_Pin, J3 Conn_01x07_Pin, J4 Conn_01x07_Pin, J5 Conn_01x07_Pin, J6 Conn_01x07_Pin, J7 Conn_01x19_MountingPin, J8 Conn_01x19_MountingPin, SW1 RotaryEncoder_Switch, SW2 RotaryEncoder_Switch

Commit message: Started new PCB design 2x3
Parts:
- moved J7 32.5 mm to (112.5, 40.8)
- moved J8 32.5 mm to (135.5, 40.8)
Routing:
- net GND: track 149.7 -> 0.00 mm
- net Key6: track 79.8 -> 0.00 mm
- net Key4: track 69.6 -> 0.00 mm
- net CS6: track 69.4 -> 0.00 mm
- net Key5: track 68.2 -> 0.00 mm
- net CS3: track 57.4 -> 0.00 mm
- net CS5: track 57.2 -> 0.00 mm
- net Key3: track 55.0 -> 0.00 mm
- net CS4: track 43.9 -> 0.00 mm
- net Key1: track 43.8 -> 0.00 mm
- net CS1: track 32.7 -> 0.00 mm
- net Key2: track 31.6 -> 0.00 mm
- net Down2: track 12.1 -> 0.00 mm
- net CS2: track 5.21 -> 0.00 mm
Other:
- board size 72 x 123.5 mm -> 74 x 155.5 mm
